File: guitar_pedal.kicad_sch (KiCad schematic)
At the start: 8 parts, among them J1 Barrel_Jack_Switch, J2 AudioJack3

Commit message: input buffer schematic added
Parts:
- added C3, C4: 22nF, symbol Device:C
- added C5: 47nF, symbol Device:C
- added Q1: Q_NPN_EBC, symbol Transistor_BJT:Q_NPN_EBC
- added R3: 1M5, symbol Device:R
- added R4: 1k, symbol Device:R
- added R5, R6: 10k, symbol Device:R
- added R7: 510k, symbol Device:R
- added R8: 4.7k, symbol Device:R
- added S1: FS57003PLT2B2M2QE, FS57003PLT2B2M2QE:SW_FS57003PLT2B2M2QE, symbol MyLabrary:FS57003PLT2B2M2QE
- added U1: NJM4558, symbol Amplifier_Operational:NJM4558
- C2: value 100uF -> 47uF
Connections:
- net +9V: now also Q1.3 (C), U1.8 (V+)
- net GND: now also R3.2, R5.1, R6.1, S1.8, U1.4 (V-)
- net Vr: now also R7.2, R8.1
- net GUITAR_IN: now reaches J2.T
- net GUITAR_IN: now also S1.1, S1.6
- new net: C5.1, R8.2
- new net: C4.2, Q1.1 (E), R5.2
- new net: Q1.2 (B), R4.2, R7.1
- new net: C3.2, R4.1
- new net +OPa_IN: C4.1, R6.2, U1.3 (+)
- new net -OPa_IN: C5.2, U1.2 (-)
- new net AMP_OUT: S1.5
- new net BYPASS_GND: S1.3, S1.9
- new net FX_IN: C3.1, R3.1, S1.2
- new net FX_OUT: S1.4
- new net LED_K: S1.7
Other:
- note added: "INPUT BUFFER"
- note added: "POWER"
- note removed: "Power"
- moved on the sheet: J2
